File: clearvideo64/clearvideo64.kicad_pcb (KiCad board)
At the start: 2 copper layers, 36 x 51.4 mm, 29 parts, among them J1 1C,2Y,3G, U1 THS7316D, U2 74F06

Commit message: Add files via upload
Parts:
- U2: value 74F06 -> 74F04
Changed lines of the file:
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@@
-(kicad_pcb (version 20171130) (host pcbnew "(5.1.2)-1")
+(kicad_pcb (version 20171130) (host pcbnew "(5.1.5)-3")
   (general
     (thickness 1.6)
@@
       (effects (font (size 1 1) (thickness 0.15)))
     )
-    (fp_text value 74F06 (at 0 5.28) (layer F.Fab) hide
-      (effects (font (size 1 1) (thickness 0.15)))
-    )
+    (fp_text value 74F04 (at 0 5.28) (layer F.Fab) hide
+      (effects (font (size 1 1) (thickness 0.15)))
+    )
