File: clearvideo64/clearvideo64.sch (KiCad schematic (older format))
At the start: 28 parts, among them J1 1C,2Y,3G, U1 THS7316D, U2 74F06

Commit message: Add files via upload
Parts:
- U2: value 74F06 -> 74F04
Connections:
- no-connect marks 0 -> 1
Changed lines of the file:
@@
 EESchema Schematic File Version 4
-LIBS:svideomod-cache
-EELAYER 29 0
+EELAYER 30 0
 EELAYER END
 $Descr A4 11693 8268
@@
 P 1050 5750
 F 0 "U2" H 1050 6067 50  0000 C CNN
-F 1 "74F06" H 1050 5976 50  0000 C CNN
+F 1 "74F04" H 1050 5976 50  0000 C CNN
 F 2 "Package_SO:SOIC-14_3.9x8.7mm_P1.27mm" H 1050 5750 50  0001 C CNN
 F 3 "http://www.ti.com/lit/gpn/sn74LS04" H 1050 5750 50  0001 C CNN
@@
 P 1050 6200
 F 0 "U2" H 1050 6517 50  0000 C CNN
-F 1 "74F06" H 1050 6426 50  0000 C CNN
+F 1 "74F04" H 1050 6426 50  0000 C CNN
 F 2 "Package_SO:SOIC-14_3.9x8.7mm_P1.27mm" H 1050 6200 50  0001 C CNN
 F 3 "http://www.ti.com/lit/gpn/sn74LS04" H 1050 6200 50  0001 C CNN
@@
 P 1050 6650
 F 0 "U2" H 1050 6967 50  0000 C CNN
-F 1 "74F06" H 1050 6876 50  0000 C CNN
+F 1 "74F04" H 1050 6876 50  0000 C CNN
 F 2 "Package_SO:SOIC-14_3.9x8.7mm_P1.27mm" H 1050 6650 50  0001 C CNN
 F 3 "http://www.ti.com/lit/gpn/sn74LS04" H 1050 6650 50  0001 C CNN
@@
 P 2900 4700
 F 0 "U2" H 2900 5017 50  0000 C CNN
-F 1 "74F06" H 2900 4926 50  0000 C CNN
+F 1 "74F04" H 2900 4926 50  0000 C CNN
 F 2 "Package_SO:SOIC-14_3.9x8.7mm_P1.27mm" H 2900 4700 50  0001 C CNN
 F 3 "http://www.ti.com/lit/gpn/sn74LS04" H 2900 4700 50  0001 C CNN
@@
 P 2900 7000
 F 0 "U2" H 2900 7317 50  0000 C CNN
-F 1 "74F06" H 2900 7226 50  0000 C CNN
+F 1 "74F04" H 2900 7226 50  0000 C CNN
 F 2 "Package_SO:SOIC-14_3.9x8.7mm_P1.27mm" H 2900 7000 50  0001 C CNN
 F 3 "http://www.ti.com/lit/gpn/sn74LS04" H 2900 7000 50  0001 C CNN
@@
 P 2900 5900
 F 0 "U2" H 2900 6217 50  0000 C CNN
-F 1 "74F06" H 2900 6126 50  0000 C CNN
+F 1 "74F04" H 2900 6126 50  0000 C CNN
 F 2 "Package_SO:SOIC-14_3.9x8.7mm_P1.27mm" H 2900 5900 50  0001 C CNN
 F 3 "http://www.ti.com/lit/gpn/sn74LS04" H 2900 5900 50  0001 C CNN
@@
 P 1100 1200
 F 0 "U2" H 1330 1246 50  0000 L CNN
-F 1 "74F06" H 1330 1155 50  0000 L CNN
+F 1 "74F04" H 1330 1155 50  0000 L CNN
 F 2 "Package_SO:SOIC-14_3.9x8.7mm_P1.27mm" H 1100 1200 50  0001 C CNN
 F 3 "http://www.ti.com/lit/gpn/sn74LS04" H 1100 1200 50  0001 C CNN
@@
 	1    0    0    -1
 $EndComp
+NoConn ~ 7150 4500
 $EndSCHEMATC
