File: clearvideo128/clearvideo128.kicad_pcb (KiCad board)
At the start: 2 copper layers, 57.8 x 45.7 mm, 47 parts, among them J3 RFM_C128, J8 AudioJack, J9 Conn_01x08, U1 74F06, U2 BA7805FP-E2, U3 LM7805_TO220, U4 THS7316D

Commit message: Add files via upload
Parts:
- removed C13, C14: 0.1, Capacitor_SMD:C_0805_2012Metric_Pad1.15x1.40mm_HandSolder
- R1, R2, R3: value 2K -> 3K3
- R5, R6, R7: value 250R -> 500R
- U1: value 74F06 -> 74F04
- moved J9 1.24 mm to (73.7, 39.2)
- renumbered AUDIO#2 to Audio#2, LUMA to J5, COLOR to J6
Connections:
- net Net-(R1-Pad1) renamed /~AEC-Y
- net Net-(R2-Pad1) renamed /~PHI-Y
- net Net-(R3-Pad1) renamed /~AEC-C
- C15 pad 2: Net-(C14-Pad2) -> Net-(C15-Pad2)
- C16 pad 2: Net-(C13-Pad1) -> Net-(C16-Pad2)
- J3 pad : (no net) -> GND
- J5 pad 2: Net-(C13-Pad2) -> Net-(C16-Pad2)
- J6 pad 2: Net-(C14-Pad1) -> Net-(C15-Pad2)
- L2 pad 2: Net-(C13-Pad1) -> Net-(C16-Pad2)
- R12 pad 1: Net-(C14-Pad2) -> Net-(C15-Pad2)
- R13 pad 1: Net-(C13-Pad1) -> Net-(C16-Pad2)
Routing:
- net Net-(C16-Pad2): track 0.00 -> 36.0 mm
- net Net-(C13-Pad2): track 22.5 -> 0.00 mm
- net /SLUM-OUT: track 78.4 -> 96.0 mm
- net Net-(C15-Pad2): track 0.00 -> 13.7 mm
- net GND: track 330.2 -> 340.8 mm
- net Net-(C13-Pad1): track 8.61 -> 0.00 mm
- net Net-(C14-Pad1): track 8.59 -> 0.00 mm
- net Net-(C14-Pad2): track 7.15 -> 0.00 mm
- net /CHR-OUT: track 67.4 -> 62.3 mm
Other:
- outline, holes or cut-outs redrawn
