File: clearvideo128/clearvideo128.sch (KiCad schematic (older format))
At the start: 47 parts, among them J1 PHCL, J2 AEC, J3 RFM_C128, J4 9V-Unreg, J5 CY, J6 CC, J7 2ndAudioChannel, J8 AudioJack, J9 Conn_01x08, U1 74F06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

Commit message: Add files via upload
Parts:
- removed C13, C14: 0.1, Capacitor_SMD:C_0805_2012Metric_Pad1.15x1.40mm_HandSolder, symbol Device:C_Small
- R1, R2, R3: value 2K -> 3K3
- R5, R6, R7: value 250R -> 500R
- U1: value 74F06 -> 74F04
Connections:
- net ~AEC-Y: now reaches R1.1, R5.1
- net ~AEC-C: now reaches R3.1, R7.1
- net ~PHI-Y: now reaches R2.1, R6.1
- net at C15.2, R12.1: now also J6.2 (Pin_2)
- net at C16.2, L2.2, R13.1: now also J5.2 (Pin_2)
- no-connect marks 8 -> 4
Changed lines of the file:
@@
 EESchema Schematic File Version 4
-LIBS:clearvideo128-cache
-EELAYER 29 0
+EELAYER 30 0
 EELAYER END
 $Descr A4 11693 8268
@@
 P 900 2400
 F 0 "U1" H 900 2717 50  0000 C CNN
-F 1 "74F06" H 900 2626 50  0000 C CNN
+F 1 "74F04" H 900 2626 50  0000 C CNN
 F 2 "Package_SO:SOIC-14_3.9x8.7mm_P1.27mm" H 900 2400 50  0001 C CNN
 F 3 "http://www.ti.com/lit/gpn/sn74LS04" H 900 2400 50  0001 C CNN
@@
 P 900 2850
 F 0 "U1" H 900 3167 50  0000 C CNN
-F 1 "74F06" H 900 3076 50  0000 C CNN
+F 1 "74F04" H 900 3076 50  0000 C CNN
 F 2 "Package_SO:SOIC-14_3.9x8.7mm_P1.27mm" H 900 2850 50  0001 C CNN
 F 3 "http://www.ti.com/lit/gpn/sn74LS04" H 900 2850 50  0001 C CNN
@@
 P 900 3300
 F 0 "U1" H 900 3617 50  0000 C CNN
-F 1 "74F06" H 900 3526 50  0000 C CNN
+F 1 "74F04" H 900 3526 50  0000 C CNN
 F 2 "Package_SO:SOIC-14_3.9x8.7mm_P1.27mm" H 900 3300 50  0001 C CNN
 F 3 "http://www.ti.com/lit/gpn/sn74LS04" H 900 3300 50  0001 C CNN
@@
 P 3150 5350
 F 0 "U1" H 3150 5667 50  0000 C CNN
-F 1 "74F06" H 3150 5576 50  0000 C CNN
+F 1 "74F04" H 3150 5576 50  0000 C CNN
 F 2 "Package_SO:SOIC-14_3.9x8.7mm_P1.27mm" H 3150 5350 50  0001 C CNN
 F 3 "http://www.ti.com/lit/gpn/sn74LS04" H 3150 5350 50  0001 C CNN
@@
 P 3150 7050
 F 0 "U1" H 3150 7367 50  0000 C CNN
-F 1 "74F06" H 3150 7276 50  0000 C CNN
+F 1 "74F04" H 3150 7276 50  0000 C CNN
 F 2 "Package_SO:SOIC-14_3.9x8.7mm_P1.27mm" H 3150 7050 50  0001 C CNN
 F 3 "http://www.ti.com/lit/gpn/sn74LS04" H 3150 7050 50  0001 C CNN
@@
 P 3150 5950
 F 0 "U1" H 3150 6267 50  0000 C CNN
-F 1 "74F06" H 3150 6176 50  0000 C CNN
+F 1 "74F04" H 3150 6176 50  0000 C CNN
 F 2 "Package_SO:SOIC-14_3.9x8.7mm_P1.27mm" H 3150 5950 50  0001 C CNN
 F 3 "http://www.ti.com/lit/gpn/sn74LS04" H 3150 5950 50  0001 C CNN
@@
 P 1100 1200
 F 0 "U1" H 1330 1246 50  0000 L CNN
-F 1 "74F06" H 1330 1155 50  0000 L CNN
+F 1 "74F04" H 1330 1155 50  0000 L CNN
 F 2 "Package_SO:SOIC-14_3.9x8.7mm_P1.27mm" H 1100 1200 50  0001 C CNN
 F 3 "http://www.ti.com/lit/gpn/sn74LS04" H 1100 1200 50  0001 C CNN
@@
 P 3550 5350
 F 0 "R1" V 3345 5350 50  0000 C CNN
-F 1 "2K" V 3436 5350 50  0000 C CNN
+F 1 "3K3" V 3436 5350 50  0000 C CNN
 F 2 "Resistor_SMD:R_0805_2012Metric_Pad1.15x1.40mm_HandSolder" H 3550 5350 50  0001 C CNN
 F 3 "~" H 3550 5350 50  0001 C CNN
@@
 P 3550 7050
 F 0 "R3" V 3345 7050 50  0000 C CNN
-F 1 "2K" V 3436 7050 50  0000 C CNN
+F 1 "3K3" V 3436 7050 50  0000 C CNN
 F 2 "Resistor_SMD:R_0805_2012Metric_Pad1.15x1.40mm_HandSolder" H 3550 7050 50  0001 C CNN
 F 3 "~" H 3550 7050 50  0001 C CNN
@@
 P 3550 5950
 F 0 "R2" V 3345 5950 50  0000 C CNN
-F 1 "2K" V 3436 5950 50  0000 C CNN
+F 1 "3K3" V 3436 5950 50  0000 C CNN
 F 2 "Resistor_SMD:R_0805_2012Metric_Pad1.15x1.40mm_HandSolder" H 3550 5950 50  0001 C CNN
 F 3 "~" H 3550 5950 50  0001 C CNN
@@
 P 4200 5500
 F 0 "R5" H 4131 5546 50  0000 R CNN
-F 1 "250R" H 4131 5455 50  0000 R CNN
+F 1 "500R" H 4131 5455 50  0000 R CNN
 F 2 "Potentiometer_THT:Potentiometer_Bourns_3296X_Horizontal" H 4200 5500 50  0001 C CNN
 F 3 "~" H 4200 5500 50  0001 C CNN
@@
 P 4200 6100
 F 0 "R6" H 4131 6146 50  0000 R CNN
-F 1 "250R" H 4131 6055 50  0000 R CNN
+F 1 "500R" H 4131 6055 50  0000 R CNN
 F 2 "Potentiometer_THT:Potentiometer_Bourns_3296X_Horizontal" H 4200 6100 50  0001 C CNN
 F 3 "~" H 4200 6100 50  0001 C CNN
@@
 P 4200 7200
 F 0 "R7" H 4131 7246 50  0000 R CNN
-F 1 "250R" H 4131 7155 50  0000 R CNN
+F 1 "500R" H 4131 7155 50  0000 R CNN
 F 2 "Potentiometer_THT:Potentiometer_Bourns_3296X_Horizontal" H 4200 7200 50  0001 C CNN
 F 3 "~" H 4200 7200 50  0001 C CNN
@@
 	7200 1200 7250 1200
 $Comp
-L Device:C_Small C13
-U 1 1 5E325728
-P 6900 1050
-F 0 "C13" V 6671 1050 50  0000 C CNN
-F 1 "0.1" V 6762 1050 50  0000 C CNN
-F 2 "Capacitor_SMD:C_0805_2012Metric_Pad1.15x1.40mm_HandSolder" H 6900 1050 50  0001 C CNN
-F 3 "~" H 6900 1050 50  0001 C CNN
-	1    6900 1050
-	0    1    1    0
-$EndComp
-$Comp
-L Device:C_Small C14
-U 1 1 5E325E1F
-P 7100 1200
-F 0 "C14" V 6900 1200 50  0000 C CNN
-F 1 "0.1" V 7000 1200 50  0000 C CNN
-F 2 "Capacitor_SMD:C_0805_2012Metric_Pad1.15x1.40mm_HandSolder" H 7100 1200 50  0001 C CNN
-F 3 "~" H 7100 1200 50  0001 C CNN
-	1    7100 1200
-	0    -1   -1   0
-$EndComp
-$Comp
 L Power2:GND #PWR019
 U 1 1 5E335C70
@@
 	1    0    0    -1
 $EndComp
-Connection ~ 7200 1200
-Wire Wire Line
-	7000 1050 7150 1050
 Wire Bus Line
 	1650 550  5350 550
@@
 	6250 900  6250 1050
 Wire Wire Line
-	6250 1050 6800 1050
-Wire Wire Line
 	6250 1350 6250 1200
-Wire Wire Line
-	6250 1200 7000 1200
 $Comp
 L Power2:GND #PWR018
@@
 Wire Wire Line
 	9800 2600 9800 2800
-NoConn ~ 9950 2400
-NoConn ~ 9950 2500
-NoConn ~ 9950 2700
-NoConn ~ 9950 3000
 NoConn ~ 10400 900
 NoConn ~ 10400 1000
+Text Label 9500 3100 0    50   ~ 0
+CHR-OUT
+Text Label 9500 2900 0    50   ~ 0
+SLUM-OUT
+Text Label 3800 5350 0    50   ~ 0
+~AEC-Y
+Text Label 3800 5950 0    50   ~ 0
+~PHI-Y
+Text Label 3800 7050 0    50   ~ 0
+~AEC-C
+Text Label 3350 4400 0    50   ~ 0
+COLOR
+Wire Wire Line
+	6250 1050 7150 1050
+Wire Wire Line
+	6250 1200 7200 1200
+Connection ~ 7200 1200
 Wire Bus Line
 	9400 2200 9400 3000
@@
 Wire Bus Line
 	1650 550  1650 4850
-Text Label 9500 3100 0    50   ~ 0
-CHR-OUT
-Text Label 9500 2900 0    50   ~ 0
-SLUM-OUT
 $EndSCHEMATC
